File: EX-CSB1.kicad_sch (KiCad schematic)
At the start: 71 parts, among them J101 MC 1,5/ 2-G-3,5, J103 MC 1,5/ 2-G-3,5, J105 STEMMA QT, J106 Conn_02x04, J107 Conn_01x10_f, J108 Conn_01x08_f, J110 MC 1,5/ 2-G-3,5, J111 Conn_01x04_f, J112 Conn_01x06_f, J113 Conn_01x08_f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

Commit message: Rev C
Removed dual I2C header to make room, Added booter common, fixed serial to conform with arduino standard, added option to provide vin_pin out by jumper (enabled by default) and added option to provide io_ref out by jumper (disabled by default).
Parts:
- removed J110: MC 1,5/ 2-G-3,5, 0_my:PhoenixContact_MC_1,5_2-G-3.5_1x02_P3.50mm_Horizontal_edited, symbol Connector_Generic:Conn_01x02
- added C121: 10u, Capacitor_SMD:C_0805_2012Metric, symbol Device:C_Small
- added J110: MC 1,5/ 3-G-3,5, Connector_Phoenix_MC:PhoenixContact_MC_1,5_3-G-3.5_1x03_P3.50mm_Horizontal, symbol Connector_Generic:Conn_01x03
- added JP103: Jumper_2, Jumper:SolderJumper-2_P1.3mm_Bridged_RoundedPad1.0x1.5mm, symbol Jumper:Jumper_2_Bridged
- added JP104: Jumper_2, Jumper:SolderJumper-2_P1.3mm_Open_RoundedPad1.0x1.5mm, symbol Jumper:Jumper_2_Open
- J106: now not fitted
Connections:
- net +3V3: now also JP104.1 (A); no longer J108.2 (Pin_2)
- net Booster-C: now also J110.2 (Pin_2)
- net Booster-D: now also J110.1 (Pin_1)
- net GND: now also C121.2, J110.3 (Pin_3)
- net USB_RX: now also J113.7 (Pin_7); no longer J113.8 (Pin_8)
- net USB_TX: now also J113.8 (Pin_8); no longer J113.7 (Pin_7)
- net VM: now also JP103.1 (A)
- net reset_n: now also C121.1
- net vin_pin: now also JP103.2 (B)
- new net io_ref: J108.2 (Pin_2), JP104.2 (B)
Other:
- moved on the sheet: C109, J107, J108, J111, J112, J113, R103
